File: midi-uart-adapter.kicad_pcb (KiCad board)
At the start: 2 copper layers, 48.3 x 61.6 mm, 25 parts, among them U1 6N138

Commit message: C2 -> C1 fix, dimensions
Parts:
- renumbered C2 to C1
Other:
- board text added: "C1 optional bridge FB1-6 if not present"
- board text removed: "C2 optional bridge FB1-6 if not present"
Changed lines of the file:
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@@
   (general
     (thickness 1.6)
-    (drawings 15)
+    (drawings 19)
     (tracks 93)
     (zones 0)
@@
     (fp_circle (center 0 0) (end 2.45 0) (layer F.CrtYd) (width 0.05))
     (fp_circle (center 0 0) (end 2.2 0) (layer Cmts.User) (width 0.15))
-    (fp_text user %R (at 0.3 0) (layer F.Fab)
+    (fp_text user %R (at 0.3 0) (layer F.Fab) hide
       (effects (font (size 1 1) (thickness 0.15)))
     )
@@
     (fp_circle (center 0 0) (end 2.45 0) (layer F.CrtYd) (width 0.05))
     (fp_circle (center 0 0) (end 2.2 0) (layer Cmts.User) (width 0.15))
-    (fp_text user %R (at 0.3 0) (layer F.Fab)
+    (fp_text user %R (at 0.3 0) (layer F.Fab) hide
       (effects (font (size 1 1) (thickness 0.15)))
     )
@@
     (tags "capacitor handsolder")
     (attr smd)
-    (fp_text reference C2 (at 0 -1.43) (layer F.SilkS)
+    (fp_text reference C1 (at 0 -1.43) (layer F.SilkS)
       (effects (font (size 1 1) (thickness 0.15)))
     )
@@
     )
   )
+  (dimension 61.595 (width 0.15) (layer F.Fab)
+    (gr_text "61.595 mm" (at 182.91 100.6475 270) (layer F.Fab)
+      (effects (font (size 1 1) (thickness 0.15)))
+    )
+    (feature1 (pts (xy 168.91 131.445) (xy 182.196421 131.445)))
+    (feature2 (pts (xy 168.91 69.85) (xy 182.196421 69.85)))
+    (crossbar (pts (xy 181.61 69.85) (xy 181.61 131.445)))
+    (arrow1a (pts (xy 181.61 131.445) (xy 181.023579 130.318496)))
+    (arrow1b (pts (xy 181.61 131.445) (xy 182.196421 130.318496)))
+    (arrow2a (pts (xy 181.61 69.85) (xy 181.023579 70.976504)))
+    (arrow2b (pts (xy 181.61 69.85) (xy 182.196421 70.976504)))
+  )
+  (dimension 55.245 (width 0.15) (layer F.Fab)
+    (gr_text "55.245 mm" (at 176.56 100.6475 90) (layer F.Fab)
+      (effects (font (size 1 1) (thickness 0.15)))
+    )
+    (feature1 (pts (xy 165.735 73.025) (xy 175.846421 73.025)))
+    (feature2 (pts (xy 165.735 128.27) (xy 175.846421 128.27)))
+    (crossbar (pts (xy 175.26 128.27) (xy 175.26 73.025)))
+    (arrow1a (pts (xy 175.26 73.025) (xy 175.846421 74.151504)))
+    (arrow1b (pts (xy 175.26 73.025) (xy 174.673579 74.151504)))
+    (arrow2a (pts (xy 175.26 128.27) (xy 175.846421 127.143496)))
+    (arrow2b (pts (xy 175.26 128.27) (xy 174.673579 127.143496)))
+  )
+  (dimension 41.91 (width 0.15) (layer F.Fab)
+    (gr_text "41.910 mm" (at 144.78 62.835) (layer F.Fab)
+      (effects (font (size 1 1) (thickness 0.15)))
+    )
+    (feature1 (pts (xy 123.825 73.025) (xy 123.825 63.548579)))
+    (feature2 (pts (xy 165.735 73.025) (xy 165.735 63.548579)))
+    (crossbar (pts (xy 165.735 64.135) (xy 123.825 64.135)))
+    (arrow1a (pts (xy 123.825 64.135) (xy 124.951504 63.548579)))
+    (arrow1b (pts (xy 123.825 64.135) (xy 124.951504 64.721421)))
+    (arrow2a (pts (xy 165.735 64.135) (xy 164.608496 63.548579)))
+    (arrow2b (pts (xy 165.735 64.135) (xy 164.608496 64.721421)))
+  )
+  (dimension 48.26 (width 0.15) (layer F.Fab)
+    (gr_text "48.260 mm" (at 144.78 57.755) (layer F.Fab)
+      (effects (font (size 1 1) (thickness 0.15)))
+    )
+    (feature1 (pts (xy 120.65 69.85) (xy 120.65 58.468579)))
+    (feature2 (pts (xy 168.91 69.85) (xy 168.91 58.468579)))
+    (crossbar (pts (xy 168.91 59.055) (xy 120.65 59.055)))
+    (arrow1a (pts (xy 120.65 59.055) (xy 121.776504 58.468579)))
+    (arrow1b (pts (xy 120.65 59.055) (xy 121.776504 59.641421)))
+    (arrow2a (pts (xy 168.91 59.055) (xy 167.783496 58.468579)))
+    (arrow2b (pts (xy 168.91 59.055) (xy 167.783496 59.641421)))
+  )
   (gr_text "Vrx = Vtx" (at 130.81 118.11) (layer F.SilkS)
     (effects (font (size 0.8 0.8) (thickness 0.15)))
   )
-  (gr_text "C2 optional\nbridge FB1-6 if not present" (at 148.59 96.52) (layer F.SilkS)
+  (gr_text "C1 optional\nbridge FB1-6 if not present" (at 148.59 96.52) (layer F.SilkS)
     (effects (font (size 0.8 0.8) (thickness 0.15)))
   )

Commit message: v2.0
Parts:
- MIDI-IN, MIDI-OUT, MIDI-THROUGH: footprint Connector_PinHeader_2.54mm:PinHeader_1x05_P2.54mm_Vertical -> Connector_PinHeader_2.54mm:PinHeader_1x03_P2.54mm_Vertical
- moved G*** 29.7 mm to (143.5, 101.6), turned to 0 degrees
- moved MIDI-IN 16.8 mm to (154.3, 92.7)
- moved REF** 15.4 mm to (158.1, 86.4)
- moved D1 14.4 mm to (140.3, 90.2), turned to 180 degrees
- moved C1 13.5 mm to (149.9, 92.7)
- moved REF** 13.3 mm to (123.8, 86.4)
- moved MIDI-THROUGH 11.8 mm to (154.3, 105.4)
- moved FB3 11.1 mm to (149.9, 97.8)
- moved FB4 11.1 mm to (149.9, 95.2)
- moved RB 10.6 mm to (144.1, 95.2)
- moved MIDI-OUT 8.64 mm to (154.3, 118.1)
- moved REF** 7.62 mm to (158.1, 128.3)
- moved FB5 7.18 mm to (149.9, 108.0)
- moved FB6 6.75 mm to (149.9, 110.5)
- moved RE 5.68 mm to (144.6, 108.0)
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Connections:
- C1 pad 1: Net-(C2-Pad1) -> Net-(C1-Pad1)
- H1 pad 3: UART_rx -> GNDREF
- H1 pad 4: UART_tx -> UART_rx
- H1 pad 5: GNDREF -> UART_tx
- MIDI-IN pad 1: Net-(MIDI-IN1-Pad1) -> Net-(C1-Pad1)
- MIDI-IN pad 2: Net-(C2-Pad1) -> Net-(FB4-Pad1)
- MIDI-IN pad 3: Net-(MIDI-IN1-Pad3) -> Net-(FB3-Pad1)
- MIDI-OUT pad 1: Net-(MIDI-OUT1-Pad1) -> GNDREF
- MIDI-OUT pad 2: GNDREF -> Net-(FB1-Pad1)
- MIDI-OUT pad 3: Net-(MIDI-OUT1-Pad3) -> Net-(FB2-Pad1)
- MIDI-THROUGH pad 1: Net-(MIDI-THROUGH1-Pad1) -> GNDREF
- MIDI-THROUGH pad 2: GNDREF -> Net-(FB5-Pad1)
- MIDI-THROUGH pad 3: Net-(MIDI-THROUGH1-Pad3) -> Net-(FB6-Pad1)
Routing:
- net GNDREF: track 112.4 -> 88.4 mm
- net Net-(D1-Pad1): track 34.0 -> 17.4 mm
- net VCC_tx: track 42.4 -> 34.8 mm
- net UART_tx: track 11.4 -> 5.28 mm
- net Net-(C2-Pad1): track 6.11 -> 0.00 mm
- net UART_rx: track 37.6 -> 31.6 mm
- net Net-(FB1-Pad1): track 6.35 -> 2.70 mm
- net Net-(C1-Pad1): track 0.00 -> 3.57 mm
- net Net-(FB1-Pad2): track 6.82 -> 3.59 mm
- net Net-(FB2-Pad1): track 6.35 -> 3.18 mm
- net Net-(D1-Pad2): track 28.4 -> 25.5 mm, vias 0 -> 1
- net Net-(FB2-Pad2): track 6.16 -> 3.33 mm
- net Net-(FB4-Pad1): track 6.11 -> 3.57 mm
- net Net-(FB3-Pad1): track 6.58 -> 4.05 mm
- net Net-(FB5-Pad1): track 6.02 -> 3.57 mm
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Other:
- board size 48.3 x 61.6 mm -> 40.6 x 48.3 mm
- board text added: "5 4 2"
- board text added: "G"
- board text added: "MIDI / UART Adapter v2.0"
- board text added: "Rx Tx"
- board text added: "Vrx Vtx"
- board text removed: "5 4 3 2 1"
- board text removed: "MIDI / UART Adapter v1.0 MIT License"
- board text removed: "Vrx Vtx Rx Tx Gnd"

Commit message: v2.1
Parts:
- moved REF** 0.64 mm to (157.5, 86.4)
- moved REF** 0.64 mm to (157.5, 128.3)
- moved REF** 0.63 mm to (124.5, 86.4)
- moved REF** 0.63 mm to (124.5, 128.3)
Other:
- board size 40.6 x 48.3 mm -> 39.4 x 48.3 mm
- board text added: "5 4 2 T R S"
- board text added: "MIDI / UART Adapter v2.1"
- board text added: "© 2020 filou.se / MIT License"
- board text removed: "5 4 2"
- board text removed: "MIDI / UART Adapter v2.0"
- board text removed: "T R S"
Changed lines of the file:
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@@
   (general
     (thickness 1.6)
-    (drawings 21)
+    (drawings 19)
     (tracks 77)
     (zones 0)
@@
       (effects (font (size 1 1) (thickness 0.15)))
     )
-    (fp_text value Conn_01x05 (at 0 7.41) (layer F.Fab)
+    (fp_text value Conn_01x05 (at 0 7.41) (layer F.Fab) hide
       (effects (font (size 1 1) (thickness 0.15)))
     )
@@
       (effects (font (size 1 1) (thickness 0.15)))
     )
-    (fp_text value Conn_01x05 (at 0 7.41) (layer F.Fab)
+    (fp_text value Conn_01x05 (at 0 7.41) (layer F.Fab) hide
       (effects (font (size 1 1) (thickness 0.15)))
     )
@@
       (effects (font (size 1 1) (thickness 0.15)))
     )
-    (fp_text value Conn_01x05 (at 0 7.41) (layer F.Fab)
+    (fp_text value Conn_01x05 (at 0 7.41) (layer F.Fab) hide
       (effects (font (size 1 1) (thickness 0.15)))
     )
@@
   )
   (module MountingHole:MountingHole_2.2mm_M2 (layer F.Cu)
-    (at 123.825 86.36)
+    (at 124.46 86.36)
     (descr "Mounting Hole 2.2mm, no annular, M2")
     (tags "mounting hole 2.2mm no annular m2")
@@
   )
   (module MountingHole:MountingHole_2.2mm_M2 (layer F.Cu)
-    (at 158.115 86.36)
+    (at 157.48 86.36)
     (descr "Mounting Hole 2.2mm, no annular, M2")
     (tags "mounting hole 2.2mm no annular m2")
@@
   )
   (module MountingHole:MountingHole_2.2mm_M2 (layer F.Cu)
-    (at 158.115 128.27)
+    (at 157.48 128.27)
     (descr "Mounting Hole 2.2mm, no annular, M2")
     (tags "mounting hole 2.2mm no annular m2")
@@
   )
   (module MountingHole:MountingHole_2.2mm_M2 (layer F.Cu)
-    (at 123.825 128.27)
+    (at 124.46 128.27)
     (descr "Mounting Hole 2.2mm, no annular, M2")
     (tags "mounting hole 2.2mm no annular m2")
@@
     (descr "Diode, DO-35_SOD27 series, Axial, Horizontal, pin pitch=10.16mm, , length*diameter=4*2mm^2, , http://www.diodes.com/_files/packages/DO-35.pdf")
     (tags "Diode DO-35_SOD27 series Axial Horizontal pin pitch 10.16mm  length 4mm diameter 2mm")
-    (fp_text reference D1 (at 5.08 1.27) (layer F.SilkS)
+    (fp_text reference D1 (at 5.08 0) (layer F.SilkS)
       (effects (font (size 1 1) (thickness 0.15)))
     )
@@
     )
   )
+  (gr_text "© 2020 filou.se / MIT License" (at 140.97 128.524) (layer F.SilkS)
+    (effects (font (size 0.9 0.9) (thickness 0.15)))
+  )
+  (dimension 39.37 (width 0.15) (layer F.Fab)
+    (gr_text "39.370 mm" (at 140.97 73.63) (layer F.Fab)
+      (effects (font (size 1 1) (thickness 0.15)))
+    )
+    (feature1 (pts (xy 121.285 83.185) (xy 121.285 74.343579)))
+    (feature2 (pts (xy 160.655 83.185) (xy 160.655 74.343579)))
+    (crossbar (pts (xy 160.655 74.93) (xy 121.285 74.93)))
+    (arrow1a (pts (xy 121.285 74.93) (xy 122.411504 74.343579)))
+    (arrow1b (pts (xy 121.285 74.93) (xy 122.411504 75.516421)))
+    (arrow2a (pts (xy 160.655 74.93) (xy 159.528496 74.343579)))
+    (arrow2b (pts (xy 160.655 74.93) (xy 159.528496 75.516421)))
+  )
+  (dimension 33.02 (width 0.15) (layer F.Fab)
+    (gr_text "33.020 mm" (at 140.97 77.44) (layer F.Fab)
+      (effects (font (size 1 1) (thickness 0.15)))
+    )
+    (feature1 (pts (xy 157.48 86.36) (xy 157.48 78.153579)))
+    (feature2 (pts (xy 124.46 86.36) (xy 124.46 78.153579)))
+    (crossbar (pts (xy 124.46 78.74) (xy 157.48 78.74)))
+    (arrow1a (pts (xy 157.48 78.74) (xy 156.353496 79.326421)))
+    (arrow1b (pts (xy 157.48 78.74) (xy 156.353496 78.153579)))
+    (arrow2a (pts (xy 124.46 78.74) (xy 125.586504 79.326421)))
+    (arrow2b (pts (xy 124.46 78.74) (xy 125.586504 78.153579)))
+  )
   (dimension 48.26 (width 0.15) (layer F.Fab)
-    (gr_text "48.260 mm" (at 172.115 107.315 270) (layer F.Fab)
-      (effects (font (size 1 1) (thickness 0.15)))
-    )
-    (feature1 (pts (xy 161.29 131.445) (xy 171.401421 131.445)))
-    (feature2 (pts (xy 161.29 83.185) (xy 171.401421 83.185)))
-    (crossbar (pts (xy 170.815 83.185) (xy 170.815 131.445)))
-    (arrow1a (pts (xy 170.815 131.445) (xy 170.228579 130.318496)))
-    (arrow1b (pts (xy 170.815 131.445) (xy 171.401421 130.318496)))
-    (arrow2a (pts (xy 170.815 83.185) (xy 170.228579 84.311504)))
-    (arrow2b (pts (xy 170.815 83.185) (xy 171.401421 84.311504)))
+    (gr_text "48.260 mm" (at 171.48 107.315 270) (layer F.Fab)
+      (effects (font (size 1 1) (thickness 0.15)))
+    )
+    (feature1 (pts (xy 160.655 131.445) (xy 170.766421 131.445)))
+    (feature2 (pts (xy 160.655 83.185) (xy 170.766421 83.185)))
+    (crossbar (pts (xy 170.18 83.185) (xy 170.18 131.445)))
+    (arrow1a (pts (xy 170.18 131.445) (xy 169.593579 130.318496)))
+    (arrow1b (pts (xy 170.18 131.445) (xy 170.766421 130.318496)))
+    (arrow2a (pts (xy 170.18 83.185) (xy 169.593579 84.311504)))
+    (arrow2b (pts (xy 170.18 83.185) (xy 170.766421 84.311504)))
   )
   (dimension 41.91 (width 0.15) (layer F.Fab)
-    (gr_text "41.910 mm" (at 167.67 107.315 270) (layer F.Fab)
-      (effects (font (size 1 1) (thickness 0.15)))
-    )
-    (feature1 (pts (xy 158.115 128.27) (xy 166.956421 128.27)))
-    (feature2 (pts (xy 158.115 86.36) (xy 166.956421 86.36)))
-    (crossbar (pts (xy 166.37 86.36) (xy 166.37 128.27)))
-    (arrow1a (pts (xy 166.37 128.27) (xy 165.783579 127.143496)))
-    (arrow1b (pts (xy 166.37 128.27) (xy 166.956421 127.143496)))
-    (arrow2a (pts (xy 166.37 86.36) (xy 165.783579 87.486504)))
-    (arrow2b (pts (xy 166.37 86.36) (xy 166.956421 87.486504)))
-  )
-  (dimension 40.64 (width 0.15) (layer F.Fab)
-    (gr_text "40.640 mm" (at 140.97 73.63) (layer F.Fab)
-      (effects (font (size 1 1) (thickness 0.15)))
-    )
-    (feature1 (pts (xy 161.29 83.185) (xy 161.29 74.343579)))
-    (feature2 (pts (xy 120.65 83.185) (xy 120.65 74.343579)))
-    (crossbar (pts (xy 120.65 74.93) (xy 161.29 74.93)))
-    (arrow1a (pts (xy 161.29 74.93) (xy 160.163496 75.516421)))
-    (arrow1b (pts (xy 161.29 74.93) (xy 160.163496 74.343579)))
-    (arrow2a (pts (xy 120.65 74.93) (xy 121.776504 75.516421)))
-    (arrow2b (pts (xy 120.65 74.93) (xy 121.776504 74.343579)))
-  )
-  (dimension 34.29 (width 0.15) (layer F.Fab)
-    (gr_text "34.290 mm" (at 140.97 77.44) (layer F.Fab)
-      (effects (font (size 1 1) (thickness 0.15)))
-    )
-    (feature1 (pts (xy 158.115 86.36) (xy 158.115 78.153579)))
-    (feature2 (pts (xy 123.825 86.36) (xy 123.825 78.153579)))
-    (crossbar (pts (xy 123.825 78.74) (xy 158.115 78.74)))
-    (arrow1a (pts (xy 158.115 78.74) (xy 156.988496 79.326421)))
-    (arrow1b (pts (xy 158.115 78.74) (xy 156.988496 78.153579)))
-    (arrow2a (pts (xy 123.825 78.74) (xy 124.951504 79.326421)))
-    (arrow2b (pts (xy 123.825 78.74) (xy 124.951504 78.153579)))
+    (gr_text "41.910 mm" (at 167.035 107.315 270) (layer F.Fab)
+      (effects (font (size 1 1) (thickness 0.15)))
+    )
+    (feature1 (pts (xy 157.48 128.27) (xy 166.321421 128.27)))
+    (feature2 (pts (xy 157.48 86.36) (xy 166.321421 86.36)))
+    (crossbar (pts (xy 165.735 86.36) (xy 165.735 128.27)))
+    (arrow1a (pts (xy 165.735 128.27) (xy 165.148579 127.143496)))
+    (arrow1b (pts (xy 165.735 128.27) (xy 166.321421 127.143496)))
+    (arrow2a (pts (xy 165.735 86.36) (xy 165.148579 87.486504)))
+    (arrow2b (pts (xy 165.735 86.36) (xy 166.321421 87.486504)))
   )
   (gr_text G (at 132.715 125.73) (layer F.SilkS)
@@
     (effects (font (size 0.9 0.9) (thickness 0.15)))
   )
-  (gr_line (start 120.65 131.445) (end 120.65 83.185) (layer Edge.Cuts) (width 0.05))
-  (gr_line (start 161.29 131.445) (end 120.65 131.445) (layer Edge.Cuts) (width 0.05))
-  (gr_line (start 161.29 83.185) (end 161.29 131.445) (layer Edge.Cuts) (width 0.05))
-  (gr_line (start 120.65 83.185) (end 161.29 83.185) (layer Edge.Cuts) (width 0.05))
-  (gr_text "T  R  S" (at 159.385 95.25 90) (layer F.SilkS)
-    (effects (font (size 1 1.025) (thickness 0.15)))
-  )
-  (gr_text "T  R  S" (at 159.385 107.95 90) (layer F.SilkS)
-    (effects (font (size 1 1.025) (thickness 0.15)))
-  )
-  (gr_text "T  R  S" (at 159.385 120.65 90) (layer F.SilkS)
-    (effects (font (size 1 1.025) (thickness 0.15)))
-  )
-  (gr_text "5  4  2" (at 157.48 95.25 90) (layer F.SilkS)
+  (gr_line (start 121.285 131.445) (end 121.285 83.185) (layer Edge.Cuts) (width 0.05))
+  (gr_line (start 160.655 131.445) (end 121.285 131.445) (layer Edge.Cuts) (width 0.05))
+  (gr_line (start 160.655 83.185) (end 160.655 131.445) (layer Edge.Cuts) (width 0.05))
+  (gr_line (start 121.285 83.185) (end 160.655 83.185) (layer Edge.Cuts) (width 0.05))
+  (gr_text "5  4  2\nT  R  S" (at 158.115 95.25 90) (layer F.SilkS)
     (effects (font (size 1 1) (thickness 0.15)))
   )
-  (gr_text "5  4  2" (at 157.48 107.95 90) (layer F.SilkS)
+  (gr_text "5  4  2\nT  R  S" (at 158.115 107.95 90) (layer F.SilkS)
     (effects (font (size 1 1) (thickness 0.15)))
   )
-  (gr_text "5  4  2" (at 157.48 123.825 90) (layer F.SilkS)
+  (gr_text "5  4  2\nT  R  S" (at 158.115 123.825 90) (layer F.SilkS)
     (effects (font (size 1 1) (thickness 0.15)) (justify left))
   )
@@
     (effects (font (size 1 0.9) (thickness 0.15)))
   )
-  (gr_text "MIDI / UART Adapter v2.0" (at 140.97 85.725) (layer F.SilkS)
+  (gr_text "MIDI / UART Adapter v2.1" (at 141.605 85.725) (layer F.SilkS)
     (effects (font (size 1 1) (thickness 0.15)))
   )
